File: Mainboard2026/MainBoard2026/MainBoard2026.kicad_sch (KiCad schematic)
At the start: 71 parts, among them J1 RJ25, J2 RJ25, J3 ICSP, J4 RJ25, J5 GPS_DFROBOT_TEL-0157, J6 Micro_SD_Card_Det_Hirose_DM3AT, J8 BATT_CON, Q4 AO3401A, SW3 POWER, U1 ESP32-WROOM-32, U2 R-78E5.0-0.5, U3 MCP25625-x-SS, U4 BP5293-33, U6 RX8900_mod, Y1 16MHz

Commit message: Add files via upload
入江さんのフィードバックを回路図に反映
Parts:
- added D2: ERR2, LED_SMD:LED_0603_1608Metric, symbol Device:LED
- added R11: 1k, Resistor_SMD:R_0603_1608Metric, symbol Device:R_US
- D20: value Zener_10V -> Zener_9V1; footprint Diode_SMD:D_SOD-323 -> KUBTSS:Zenner
- D4: value SCK -> SD
- D5: value ERR -> CAN
- D6: value BATT -> ERR
- R5, R6: value 1k -> 2k
Connections:
- net +3V3: now also D4.2 (A), D5.2 (A), J5.1 (Pin_1), R25.2
- net +5V: no longer J5.1 (Pin_1)
- net CS: now also R6.2, U1.23 (IO15); no longer U1.9 (IO33)
- net CS1: now also R5.2
- net DET: now also U1.6 (IO34); no longer U1.36 (IO22)
- net ERR: now also D6.2 (A), U1.11 (IO26); no longer D5.2 (A), U1.7 (IO35)
- net GND: now also R11.2; no longer R25.2, R5.2, R6.2
- net INT: now also U1.26 (IO4); no longer U1.8 (IO32)
- net MISO: now also U1.31 (IO19); no longer U1.33 (IO21)
- net SCL: now also U1.36 (IO22); no longer U1.13 (IO14)
- net SDA: now also U1.33 (IO21); no longer U1.23 (IO15)
- net TX1: now also U1.28 (IO17); no longer U1.26 (IO4)
- net at C7.1, R27.2: now also U1.7 (IO35); no longer U1.29 (IO5)
- net at R31.1: now also U1.37 (IO23); no longer U1.30 (IO18)
- net ERR2: now reaches U1.12 (IO27)
- net ERR2: now also D2.2 (A)
- net at R30.1: now also U1.29 (IO5); no longer U1.28 (IO17)
- net at R32.1: now also U1.30 (IO18); no longer U1.31 (IO19)
- removed net BAT: D6.2 (A), U1.6 (IO34)
- net LED1: no longer names the net of U1.10 (IO25)
- net LED1: no longer D4.2 (A)
- new net: D2.1 (K), R11.1
Other:
- note added: "I2C SDA:IO21,SCL:IO22 SPI SCK:IO18,MISO:IO19,MOSI:IO23,CS:IO5, CS2:IO15 UART0(書き込み） TX:IO1,RX:IO3 UART1(未接続） UART2(外部機器） TX:IO17,RX16"
- moved on the sheet: C7, D4, D5, D6, J3, JP1, R25, R27, R30, R31, R32, R5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
