File: MainBoard2026/MainBoard2026.kicad_pcb (KiCad board)
At the start: 2 copper layers, 47 parts, among them J1 RJ25, J2 RJ25, J3 BATT_CON, J4 PRG_TWE, J5 GPS_DFROBOT_TEL-0157, J6 Micro_SD_Card_Det_Hirose_DM3AT, J7 RJ25, Q1 Q_PMOS_GDS, SW3 SW_Push, SW4 REG, U2 R-78E5.0-0.5, U3 MCP25625-x-SS, U6 RX8900_mod, U7 TWE-L-WX, Y1 16MHz

Commit message: Add files via upload
フットプリント設定完了
Parts:
- removed D3: SK54, Diode_SMD:D_SMC
- removed J3: BATT_CON, Connector_AMASS:AMASS_XT60PW-M_1x02_P7.20mm_Horizontal
- removed J7: RJ25, Connector_RJ:RJ25_Wayconn_MJEA-660X1_Horizontal
- removed JP2: M1, Jumper:SolderJumper-2_P1.3mm_Open_RoundedPad1.0x1.5mm
- removed JP3: BPS, Jumper:SolderJumper-2_P1.3mm_Open_RoundedPad1.0x1.5mm
- removed JP4: TX, Connector_PinHeader_2.54mm:PinHeader_1x02_P2.54mm_Vertical
- removed JP5: RX, Connector_PinHeader_2.54mm:PinHeader_1x02_P2.54mm_Vertical
- removed Q1: Q_PMOS_GDS, Package_TO_SOT_SMD:TO-252-2
- removed SW4: REG, Button_Switch_SMD:SW_SPST_PTS810
- removed U7: TWE-L-WX, RF_Module:MonoWireless_TWE-L-WX
- added C13: 10u, Capacitor_SMD:C_0603_1608Metric, F.Cu at (46.3, 77.8)
- added C14: 0.1u, Capacitor_SMD:C_0603_1608Metric, F.Cu at (46.3, 80.3)
- added C15: 1u, Capacitor_SMD:C_0603_1608Metric, F.Cu at (46.3, 82.8)
- added C16: 0.1u, Capacitor_SMD:C_0603_1608Metric, F.Cu at (50.3, 62.7)
- added C17: 100u, Capacitor_SMD:C_1206_3216Metric, F.Cu at (60.3, 102.5)
- added C21: 1u, Capacitor_SMD:C_0603_1608Metric, F.Cu at (50.3, 65.2)
- added C22: 22u, Capacitor_SMD:C_0603_1608Metric, F.Cu at (50.3, 67.7)
- added C23: 0.1u, Capacitor_SMD:C_0603_1608Metric, F.Cu at (50.3, 70.2)
- added C24: 0.1u, Capacitor_SMD:C_0603_1608Metric, F.Cu at (50.3, 72.8)
- added C25: 22u, Capacitor_SMD:C_0603_1608Metric, F.Cu at (50.3, 75.3)
- added C26: 22u, Capacitor_SMD:C_0603_1608Metric, F.Cu at (50.3, 77.8)
- added C27: 0.1u, Capacitor_SMD:C_0603_1608Metric, F.Cu at (50.3, 80.3)
- added C28: 0.1u, Capacitor_SMD:C_0603_1608Metric, F.Cu at (50.3, 82.8)
- added C29: 22u, Capacitor_SMD:C_0603_1608Metric, F.Cu at (54.3, 62.7)
- added C5: 10u, Capacitor_SMD:C_1206_3216Metric, F.Cu at (60.3, 99.1)
- added C8: 0.1u, Capacitor_SMD:C_0603_1608Metric, F.Cu at (46.3, 75.3)
- added D20: Zener_10V, Diode_SMD:D_SOD-323, F.Cu at (89.7, 43.8)
- added F2: MF-R090, KUBTSS:Fuse MF-R090, F.Cu at (89.4, 49.0)
- added FB1: FerriteBead_Small, Inductor_SMD:L_0603_1608Metric, F.Cu at (54.3, 65.2)
- added J8: BATT_CON, Connector_AMASS:AMASS_XT60PW-M_1x02_P7.20mm_Horizontal, F.Cu at (69.5, 102.5)
- added Q4: AO3401A, Package_TO_SOT_SMD:SOT-23, F.Cu at (90.0, 36.2)
- added R19: 100k, Resistor_SMD:R_0603_1608Metric, F.Cu at (58.3, 75.3)
- added R20: 22, Resistor_SMD:R_0603_1608Metric, F.Cu at (58.3, 77.8)
- added R21: 33, Resistor_SMD:R_0603_1608Metric, F.Cu at (58.3, 80.3)
- added R23: 100k, Resistor_SMD:R_0603_1608Metric, F.Cu at (58.3, 82.8)
- added R25: 100k, Resistor_SMD:R_0603_1608Metric, F.Cu at (62.3, 62.7)
- added R26: 200k, Resistor_SMD:R_0603_1608Metric, F.Cu at (62.3, 65.2)
- added R27: 100k, Resistor_SMD:R_0603_1608Metric, F.Cu at (62.3, 67.7)
- added R30: 33, Resistor_SMD:R_0603_1608Metric, F.Cu at (62.3, 70.2)
- added R31: 33, Resistor_SMD:R_0603_1608Metric, F.Cu at (62.3, 72.8)
- added R32: 33, Resistor_SMD:R_0603_1608Metric, F.Cu at (62.3, 75.3)
- added R42: 100k, Resistor_SMD:R_0603_1608Metric, F.Cu at (62.3, 77.8)
- added R44: 4.7k, Resistor_SMD:R_0603_1608Metric, F.Cu at (62.3, 80.3)
- added U1: ESP32-WROOM-32, RF_Module:ESP32-WROOM-32, F.Cu at (52.5, 50.4)
- added U4: R-78E3.3-0.5, Converter_DCDC:Converter_DCDC_RECOM_R-78E-0.5_THT, F.Cu at (48.5, 101.5)
- added U5: ~, KUBTSS:BNO055, F.Cu at (83.3, 67.2)
- C2: value 0.1u -> 10u
- C3: value 0.1u -> 1u
- D9: value IM920 -> RB160M; footprint LED_SMD:LED_0603_1608Metric -> Diode_SMD:D_SOD-123
- J4: value PRG_TWE -> RJ25; footprint Connector_PinSocket_2.54mm:PinSocket_1x06_P2.54mm_Vertical -> Connector_RJ:RJ25_Wayconn_MJEA-660X1_Horizontal
- R10: value 1k -> 330k
- R12: value 1k -> 47k
- R4: value 20k -> 100k
- R8: value 10k -> 22
- SW3: value SW_Push -> POWER; footprint Button_Switch_SMD:SW_SPST_PTS810 -> KUBTSS:toggle
- moved Y1 71.4 mm to (90.1, 40.2)
- moved J4 71.1 mm to (38.7, 94.7)
- moved D10 58.4 mm to (60.4, 95.8)
- moved BT1 55.5 mm to (91.1, 89.3)
- moved D7 55.4 mm to (60.4, 89.1)
- moved D1 55.4 mm to (60.4, 85.7)
- moved SW3 51.5 mm to (85.1, 98.2)
- moved U3 48.7 mm to (82.3, 39.8)
- moved J5 42.5 mm to (80.5, 23.6)
- moved U2 39.6 mm to (48.5, 91.3)
- moved JP1 37.1 mm to (90.0, 58.7)
- moved D4 35.5 mm to (90.2, 94.8)
- moved D5 35.5 mm to (90.2, 97.4)
- moved D8 35.5 mm to (90.2, 102.6)
- moved D6 35.5 mm to (90.2, 100.0)
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Connections:
- C2 pad 1: GND -> Net-(U3-VDDA)
- C2 pad 2: +3V3 -> GND
- C3 pad 1: +3V3 -> +5V
- C4 pad 1: +5V -> Net-(U3-VDDA)
- C7 pad 1: VSENS -> Net-(U1-IO5)
- D10 pad 2: VSENS -> Net-(D10-A)
- D4 pad 2: SCK -> LED1
- D8 pad 2: SCK -> LED2
- D9 pad 1: Net-(D9-K) -> +BATT
- D9 pad 2: LED_IM920 -> +3.3V
- J4 pad 1: GND -> unconnected-(J4-Pad1)
- J4 pad 2: TXD_TWE -> GND
- J4 pad 3: PRG_TWE -> CAN_L
- J4 pad 4: RXD_TWE -> CAN_H
- J4 pad 5: RST_TWE -> +BATT
- J4 pad 6: +3V3 -> unconnected-(J4-Pad6)
- J6 pad 1: unconnected-(J6-DAT2-Pad1) -> Net-(J6-DAT1)
- J6 pad 11: unconnected-(J6-SHIELD-Pad11) -> GND
- J6 pad 7: MISO -> Net-(J6-DAT0)
- J6 pad 8: unconnected-(J6-DAT1-Pad8) -> Net-(J6-DAT1)
- R12 pad 1: Net-(D9-K) -> CS1
- R12 pad 2: GND -> +3V3
- R4 pad 1: Net-(D3-K) -> +3V3
- R4 pad 2: Net-(Q1-G) -> MOSI
- R8 pad 1: Net-(Q1-G) -> Net-(J6-DAT0)
- R8 pad 2: GND -> MISO
- SW3 pad 1: Net-(U4-RUN) -> GND
- SW3 pad 2: GND -> Net-(SW3-B)
- U3 pad 17: CS -> Net-(U3-~{CS})
- U3 pad 19: +3V3 -> +5V
- U3 pad 27: +5V -> Net-(U3-VDDA)
- U3 pad 5: GND -> Net-(U3-STBY)

Commit message: Add files via upload
Parts:
- removed D8: SPI, LED_SMD:LED_0603_1608Metric
- removed R11: 1k, Resistor_SMD:R_0603_1608Metric
- removed R20: 22, Resistor_SMD:R_0603_1608Metric
- removed R21: 33, Resistor_SMD:R_0603_1608Metric
- added J3: ICSP, Connector_PinHeader_2.54mm:PinHeader_2x03_P2.54mm_Vertical, F.Cu at (157.4, 49.9)
- added R13: 10k, Resistor_SMD:R_0603_1608Metric, B.Cu at (165.6, 64.3)
- added REF**: MountingHole_4.3mm_M4, MountingHole:MountingHole_4.3mm_M4, F.Cu at (200.0, 79.8)
- added REF**: MountingHole_4.3mm_M4, MountingHole:MountingHole_4.3mm_M4, F.Cu at (149.6, 94.4)
- added REF**: MountingHole_4.3mm_M4, MountingHole:MountingHole_4.3mm_M4, F.Cu at (149.6, 49.2)
- BT1, C13, C14, C15, C16, C17, C2, C21, C22, C23, C24, C25, C26, C27, C28, C29, C3, C4, C6, C7, C8, D1, D10, D20, D7, D9, FB1, JP1, Q4, R1, R10, R12, R19, R2, R23, R25, R26, R27, R3, R30, R31, R32, R4, R42, R44, R8, R9, U3, Y1: moved to B.Cu
- C5: footprint Capacitor_SMD:C_1206_3216Metric -> Capacitor_SMD:C_0603_1608Metric; moved to B.Cu
- U1: footprint RF_Module:ESP32-WROOM-32 -> KUBTSS:ESP32-WROOM-32
- U4: value R-78E3.3-0.5 -> BP5293-33; footprint Converter_DCDC:Converter_DCDC_RECOM_R-78E-0.5_THT -> KUBTSS:BP5293-33
- moved J4 157.4 mm to (195.9, 87.9)
- moved C2 147.8 mm to (193.1, 79.5)
- moved C3 147.6 mm to (193.6, 74.4)
- moved C14 147.5 mm to (193.6, 72.9)
- moved C4 147.2 mm to (193.1, 78.0)
- moved C13 145.3 mm to (189.6, 53.9), turned to 90 degrees
- moved C22 143.8 mm to (193.5, 81.7), turned to -90 degrees
- moved C6 142.8 mm to (188.1, 53.9), turned to 90 degrees
- moved J2 141.7 mm to (180.2, 87.8)
- moved C23 140.7 mm to (190.6, 80.9)
- moved FB1 139.2 mm to (193.1, 76.5), turned to 180 degrees
- moved U2 138.6 mm to (186.7, 82.6)
- moved R4 138.1 mm to (190.3, 51.6), turned to 180 degrees
- moved C24 137.5 mm to (187.6, 80.8), turned to 180 degrees
- moved C7 136.6 mm to (182.1, 58.0), turned to -90 degrees
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Connections:
- C28 pad 2: +3.3V -> +3V3
- C29 pad 2: +3.3V -> +3V3
- D9 pad 2: +3.3V -> +3V3
- Q4 pad 2: +out -> +BATT
- R25 pad 1: unconnected-(R25-Pad1) -> TX1
- U1 pad 11: LED2 -> unconnected-(U1-IO26-Pad11)
- U1 pad 12: TX1 -> unconnected-(U1-IO27-Pad12)
- U1 pad 14: unconnected-(U1-IO12-Pad14) -> Net-(U1-IO12)
- U1 pad 26: unconnected-(U1-IO4-Pad26) -> TX1
- U1 pad 9: Net-(U1-IO33) -> CS
- U3 pad 17: Net-(U3-~{CS}) -> CS
- U4 pad 3: +3.3V -> +3V3
Routing:
- net +3V3: track 0.00 -> 101.5 mm, vias 0 -> 3
- net +BATT: track 0.00 -> 91.8 mm, vias 0 -> 1
- net CAN_H: track 0.00 -> 61.1 mm, vias 0 -> 1
- net GND: track 0.00 -> 56.3 mm, vias 0 -> 38
- net CAN_L: track 0.00 -> 49.3 mm, vias 0 -> 1
- net CS: track 0.00 -> 31.7 mm, vias 0 -> 1
- net IO0: track 0.00 -> 30.3 mm, vias 0 -> 3
- net INT: track 0.00 -> 27.4 mm, vias 0 -> 1
- net TX: track 0.00 -> 27.3 mm, vias 0 -> 1
- net RX: track 0.00 -> 26.2 mm, vias 0 -> 1
- net MISO: track 0.00 -> 23.6 mm, vias 0 -> 2
- net +5V: track 0.00 -> 22.7 mm
- net MOSI: track 0.00 -> 22.0 mm, vias 0 -> 3
- net DET: track 0.00 -> 21.3 mm
- net SDA: track 0.00 -> 20.1 mm
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- added copper zone on B.Cu, net GND
- added copper zone on F.Cu, net GND
Other:
- board outline added: 60 x 55.4 mm
