File: MainBoard2026/MainBoard2026.kicad_pcb (KiCad board)
At the start: 2 copper layers, 60 x 55.4 mm, 74 parts, among them J1 RJ25, J2 RJ25, J3 ICSP, J4 RJ25, J5 GPS_DFROBOT_TEL-0157, J6 Micro_SD_Card_Det_Hirose_DM3AT, J8 BATT_CON, Q4 AO3401A, SW3 POWER, U1 ESP32-WROOM-32, U2 R-78E5.0-0.5, U3 MCP25625-x-SS, U4 BP5293-33, U6 RX8900_mod, Y1 16MHz

Commit message: Add files via upload
Parts:
- removed BT1: MS621FE FL11E, Battery:BatteryHolder_Seiko_MS621F
- removed C13, C2, C5: 10u, Capacitor_SMD:C_0603_1608Metric
- removed C14, C16, C23, C24, C27, C28, C4, C6, C7, C8: 0.1u, Capacitor_SMD:C_0603_1608Metric
- removed C15, C21, C3: 1u, Capacitor_SMD:C_0603_1608Metric
- removed C17: 100u, Capacitor_SMD:C_1206_3216Metric
- removed C22, C25, C26, C29: 22u, Capacitor_SMD:C_0603_1608Metric
- removed D1, D10, D7, D9: RB160M, Diode_SMD:D_SOD-123
- removed D20: Zener_10V, Diode_SMD:D_SOD-323
- removed D4: SCK, LED_SMD:LED_0603_1608Metric
- removed D5: ERR, LED_SMD:LED_0603_1608Metric
- removed D6: BATT, LED_SMD:LED_0603_1608Metric
- removed F2: MF-R090, KUBTSS:Fuse MF-R090
- removed FB1: FerriteBead_Small, Inductor_SMD:L_0603_1608Metric
- removed J1, J2, J4: RJ25, Connector_RJ:RJ25_Wayconn_MJEA-660X1_Horizontal
- removed J3: ICSP, Connector_PinHeader_2.54mm:PinHeader_2x03_P2.54mm_Vertical
- removed J5: GPS_DFROBOT_TEL-0157, Connector_JST:JST_XA_S04B-XASK-1_1x04_P2.50mm_Horizontal
- removed J6: Micro_SD_Card_Det_Hirose_DM3AT, Connector_Card:microSD_HC_Hirose_DM3AT-SF-PEJM5
- removed J8: BATT_CON, Connector_AMASS:AMASS_XT60PW-M_1x02_P7.20mm_Horizontal
- removed JP1: Terminate, Jumper:SolderJumper-2_P1.3mm_Open_RoundedPad1.0x1.5mm
- removed Q4: AO3401A, Package_TO_SOT_SMD:SOT-23
- removed R1, R13, R3: 10k, Resistor_SMD:R_0603_1608Metric
- removed R10: 330k, Resistor_SMD:R_0603_1608Metric
- removed R12: 47k, Resistor_SMD:R_0603_1608Metric
- removed R19, R23, R25, R27, R4, R42: 100k, Resistor_SMD:R_0603_1608Metric
- removed R2, R5, R6, R7: 1k, Resistor_SMD:R_0603_1608Metric
- removed R26: 200k, Resistor_SMD:R_0603_1608Metric
- removed R30, R31, R32: 33, Resistor_SMD:R_0603_1608Metric
- removed R44: 4.7k, Resistor_SMD:R_0603_1608Metric
- removed R8: 22, Resistor_SMD:R_0603_1608Metric
- removed R9: 120, Resistor_SMD:R_0603_1608Metric
- removed REF** (x3): MountingHole_4.3mm_M4, MountingHole:MountingHole_4.3mm_M4
- removed SW3: POWER, KUBTSS:toggle
- removed U1: ESP32-WROOM-32, KUBTSS:ESP32-WROOM-32
- removed U2: R-78E5.0-0.5, Converter_DCDC:Converter_DCDC_RECOM_R-78E-0.5_THT
- removed U3: MCP25625-x-SS, Package_SO:SSOP-28_5.3x10.2mm_P0.65mm
- removed U4: BP5293-33, KUBTSS:BP5293-33
- removed U5: ~, KUBTSS:BNO055
- removed U6: RX8900_mod, Package_DIP:DIP-8_W7.62mm
- removed Y1: 16MHz, Crystal:Resonator_SMD_Murata_CSTxExxV-3Pin_3.0x1.1mm
Routing:
- net +3V3: track 101.5 -> 0.00 mm, vias 3 -> 0
- net +BATT: track 91.8 -> 0.00 mm, vias 1 -> 0
- net CAN_H: track 61.1 -> 0.00 mm, vias 1 -> 0
- net GND: track 56.3 -> 0.00 mm, vias 38 -> 0
- net CAN_L: track 49.3 -> 0.00 mm, vias 1 -> 0
- net CS: track 31.7 -> 0.00 mm, vias 1 -> 0
- net IO0: track 30.3 -> 0.00 mm, vias 3 -> 0
- net INT: track 27.4 -> 0.00 mm, vias 1 -> 0
- net TX: track 27.3 -> 0.00 mm, vias 1 -> 0
- net RX: track 26.2 -> 0.00 mm, vias 1 -> 0
- net MISO: track 23.6 -> 0.00 mm, vias 2 -> 0
- net +5V: track 22.7 -> 0.00 mm
- net MOSI: track 22.0 -> 0.00 mm, vias 3 -> 0
- net DET: track 21.3 -> 0.00 mm
- net SDA: track 20.1 -> 0.00 mm
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- removed copper zone on B.Cu, net GND
- removed copper zone on F.Cu, net GND
Other:
- board outline removed

Commit message: Add files via upload
Parts:
- added BT1: MS621FE FL11E, Battery:BatteryHolder_Seiko_MS621F, F.Cu at (84.0, 65.6)
- added C13: 10u, Capacitor_SMD:C_0603_1608Metric, F.Cu at (40.0, 80.2)
- added C14: 0.1u, Capacitor_SMD:C_0603_1608Metric, F.Cu at (40.0, 82.7)
- added C15: 1u, Capacitor_SMD:C_0603_1608Metric, F.Cu at (44.0, 62.6)
- added C16: 0.1u, Capacitor_SMD:C_0603_1608Metric, F.Cu at (44.0, 65.1)
- added C17: 100u, Capacitor_SMD:C_1206_3216Metric, F.Cu at (83.4, 81.1)
- added C2: 10u, Capacitor_SMD:C_0603_1608Metric, F.Cu at (40.0, 62.6)
- added C21: 1u, Capacitor_SMD:C_0603_1608Metric, F.Cu at (44.0, 67.6)
- added C22: 22u, Capacitor_SMD:C_0603_1608Metric, F.Cu at (44.0, 70.1)
- added C23: 0.1u, Capacitor_SMD:C_0603_1608Metric, F.Cu at (44.0, 72.6)
- added C24: 0.1u, Capacitor_SMD:C_0603_1608Metric, F.Cu at (44.0, 75.2)
- added C25: 22u, Capacitor_SMD:C_0603_1608Metric, F.Cu at (44.0, 77.7)
- added C26: 22u, Capacitor_SMD:C_0603_1608Metric, F.Cu at (44.0, 80.2)
- added C27: 0.1u, Capacitor_SMD:C_0603_1608Metric, F.Cu at (44.0, 82.7)
- added C28: 0.1u, Capacitor_SMD:C_0603_1608Metric, F.Cu at (48.0, 62.6)
- added C29: 22u, Capacitor_SMD:C_0603_1608Metric, F.Cu at (48.0, 65.1)
- added C3: 1u, Capacitor_SMD:C_0603_1608Metric, F.Cu at (40.0, 65.1)
- added C4: 0.1u, Capacitor_SMD:C_0603_1608Metric, F.Cu at (40.0, 67.6)
- added C5: 10u, Capacitor_SMD:C_0603_1608Metric, F.Cu at (40.0, 70.1)
- added C6: 0.1u, Capacitor_SMD:C_0603_1608Metric, F.Cu at (40.0, 72.6)
- added C7: 0.1u, Capacitor_SMD:C_0603_1608Metric, F.Cu at (40.0, 75.2)
- added C8: 0.1u, Capacitor_SMD:C_0603_1608Metric, F.Cu at (40.0, 77.7)
- added D1: RB160M, Diode_SMD:D_SOD-123, F.Cu at (77.7, 71.4)
- added D10: RB160M, Diode_SMD:D_SOD-123, F.Cu at (77.7, 81.5)
- added D2: ERR2, LED_SMD:LED_0603_1608Metric, F.Cu at (83.5, 39.1)
- added D20: Zener_9V1, KUBTSS:Zenner, F.Cu at (54.1, 85.0)
- added D4: SD, LED_SMD:LED_0603_1608Metric, F.Cu at (83.5, 41.7)
- added D5: CAN, LED_SMD:LED_0603_1608Metric, F.Cu at (83.5, 44.3)
- added D6: ERR, LED_SMD:LED_0603_1608Metric, F.Cu at (83.5, 46.9)
- added D7: RB160M, Diode_SMD:D_SOD-123, F.Cu at (77.7, 74.8)
- added D9: RB160M, Diode_SMD:D_SOD-123, F.Cu at (77.7, 78.1)
- added F2: MF-R090, KUBTSS:Fuse MF-R090, F.Cu at (87.1, 40.9)
- added FB1: FerriteBead_Small, Inductor_SMD:L_0603_1608Metric, F.Cu at (48.0, 67.6)
- added J1: RJ25, Connector_RJ:RJ25_Wayconn_MJEA-660X1_Horizontal, F.Cu at (32.4, 64.5)
- added J2: RJ25, Connector_RJ:RJ25_Wayconn_MJEA-660X1_Horizontal, F.Cu at (32.4, 79.6)
- added J3: ICSP, Connector_PinHeader_2.54mm:PinHeader_2x03_P2.54mm_Vertical, F.Cu at (82.9, 72.1)
- added J4: RJ25, Connector_RJ:RJ25_Wayconn_MJEA-660X1_Horizontal, F.Cu at (32.4, 94.6)
- added J5: GPS_DFROBOT_TEL-0157, Connector_JST:JST_XA_S04B-XASK-1_1x04_P2.50mm_Horizontal, F.Cu at (41.5, 88.4)
- added J6: Micro_SD_Card_Det_Hirose_DM3AT, Connector_Card:microSD_HC_Hirose_DM3AT-SF-PEJM5, F.Cu at (66.4, 70.7)
- added J8: BATT_CON, Connector_AMASS:AMASS_XT60PW-M_1x02_P7.20mm_Horizontal, F.Cu at (63.2, 102.3)
- added JP1: Terminate, Jumper:SolderJumper-2_P1.3mm_Open_RoundedPad1.0x1.5mm, F.Cu at (86.1, 33.4)
- added Q4: AO3401A, Package_TO_SOT_SMD:SOT-23, F.Cu at (55.0, 96.4)
- added R1: 10k, Resistor_SMD:R_0603_1608Metric, F.Cu at (48.0, 70.1)
- added R10: 330k, Resistor_SMD:R_0603_1608Metric, F.Cu at (52.0, 70.1)
- added R11: 1k, Resistor_SMD:R_0603_1608Metric, F.Cu at (52.0, 72.6)
- added R12: 47k, Resistor_SMD:R_0603_1608Metric, F.Cu at (52.0, 75.2)
- added R13: 10k, Resistor_SMD:R_0603_1608Metric, F.Cu at (52.0, 77.7)
- added R19: 100k, Resistor_SMD:R_0603_1608Metric, F.Cu at (52.0, 80.2)
- added R2: 1k, Resistor_SMD:R_0603_1608Metric, F.Cu at (48.0, 72.6)
- added R23: 100k, Resistor_SMD:R_0603_1608Metric, F.Cu at (52.0, 82.7)
- added R25: 100k, Resistor_SMD:R_0603_1608Metric, F.Cu at (56.0, 62.6)
- added R26: 200k, Resistor_SMD:R_0603_1608Metric, F.Cu at (56.0, 65.1)
- added R27: 100k, Resistor_SMD:R_0603_1608Metric, F.Cu at (56.0, 67.6)
- added R3: 10k, Resistor_SMD:R_0603_1608Metric, F.Cu at (48.0, 75.2)
- added R30: 33, Resistor_SMD:R_0603_1608Metric, F.Cu at (56.0, 70.1)
- added R31: 33, Resistor_SMD:R_0603_1608Metric, F.Cu at (56.0, 72.6)
- added R32: 33, Resistor_SMD:R_0603_1608Metric, F.Cu at (56.0, 75.2)
- added R4: 100k, Resistor_SMD:R_0603_1608Metric, F.Cu at (48.0, 77.7)
- added R42: 100k, Resistor_SMD:R_0603_1608Metric, F.Cu at (56.0, 77.7)
- added R44: 4.7k, Resistor_SMD:R_0603_1608Metric, F.Cu at (56.0, 80.2)
- added R5: 2k, Resistor_SMD:R_0603_1608Metric, F.Cu at (48.0, 80.2)
- added R6: 2k, Resistor_SMD:R_0603_1608Metric, F.Cu at (48.0, 82.7)
- added R7: 1k, Resistor_SMD:R_0603_1608Metric, F.Cu at (52.0, 62.6)
- added R8: 22, Resistor_SMD:R_0603_1608Metric, F.Cu at (52.0, 65.1)
- added R9: 120, Resistor_SMD:R_0603_1608Metric, F.Cu at (52.0, 67.6)
- added SW3: POWER, KUBTSS:toggle, F.Cu at (84.4, 54.2)
- added U1: ESP32-WROOM-32, KUBTSS:ESP32-WROOM-32, F.Cu at (46.2, 50.3)
- added U2: R-78E5.0-0.5, Converter_DCDC:Converter_DCDC_RECOM_R-78E-0.5_THT, F.Cu at (74.9, 35.0)
- added U3: MCP25625-x-SS, Package_SO:SSOP-28_5.3x10.2mm_P0.65mm, F.Cu at (75.9, 55.4)
- added U4: BP5293-33, KUBTSS:BP5293-33, F.Cu at (79.9, 25.2)
- added U5: ~, KUBTSS:BNO055, F.Cu at (77.8, 90.7)
- added U6: RX8900_mod, Package_DIP:DIP-8_W7.62mm, F.Cu at (72.3, 39.9)
- added Y1: 16MHz, Crystal:Resonator_SMD_Murata_CSTxExxV-3Pin_3.0x1.1mm, F.Cu at (86.5, 29.4)
