File: MainBoard2026/MainBoard2026.kicad_pcb (KiCad board)
At the start: 2 copper layers, 73 parts, among them J1 RJ25, J2 RJ25, J3 ICSP, J4 RJ25, J5 GPS_DFROBOT_TEL-0157, J6 Micro_SD_Card_Det_Hirose_DM3AT, J8 BATT_CON, Q4 AO3401A, SW3 POWER, U1 ESP32-WROOM-32, U2 R-78E5.0-0.5, U3 MCP25625-x-SS, U4 BP5293-33, U6 RX8900_mod, Y1 16MHz

Commit message: Add files via upload
Parts:
- C13, C14, C15, C16, C17, C2, C21, C22, C23, C24, C25, C26, C27, C28, C29, C3, C4, C5, C6, C7, C8, D1, D10, D7, D9, F2, FB1, J3, JP1, Q4, R1, R10, R11, R12, R13, R19, R2, R23, R25, R26, R27, R3, R30, R31, R32, R4, R42, R44, R5, R6, R7, R8, R9, Y1: moved to B.Cu
- moved J1 129.4 mm to (160.6, 82.4)
- moved J5 118.9 mm to (156.4, 57.6), turned to 90 degrees
- moved J2 112.9 mm to (145.2, 82.4)
- moved C27 112.7 mm to (153.1, 54.4), turned to -90 degrees
- moved R10 110.7 mm to (156.1, 32.3), turned to 180 degrees
- moved C26 110.6 mm to (151.6, 54.4), turned to -90 degrees
- moved C28 105.7 mm to (153.1, 51.4), turned to 90 degrees
- moved C29 104.5 mm to (151.6, 51.4), turned to 90 degrees
- moved J4 98.3 mm to (129.9, 82.4)
- moved R5 98.3 mm to (138.2, 41.2), turned to 180 degrees
- moved C22 98.1 mm to (142.1, 71.5)
- moved C23 98.1 mm to (142.1, 73.0)
- moved C8 97.9 mm to (124.8, 28.7), turned to 90 degrees
- moved U5 96.9 mm to (156.6, 34.2)
- moved C21 96.5 mm to (140.5, 65.6), turned to -90 degrees
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Connections:
- U3 pad 26: unconnected-(U3-VSS-Pad26) -> GND
Routing:
- net +3V3: track 0.00 -> 145.8 mm, vias 0 -> 8
- net +BATT: track 0.00 -> 91.3 mm, vias 0 -> 1
- net GND: track 0.00 -> 80.6 mm, vias 0 -> 84
- net VSENS: track 0.00 -> 77.2 mm
- net INT: track 0.00 -> 64.1 mm, vias 0 -> 4
- net MOSI: track 0.00 -> 49.5 mm, vias 0 -> 1
- net CAN_H: track 0.00 -> 48.5 mm
- net SCK: track 0.00 -> 45.4 mm, vias 0 -> 4
- net CAN_L: track 0.00 -> 45.4 mm, vias 0 -> 1
- net MISO: track 0.00 -> 37.8 mm, vias 0 -> 5
- net CS1: track 0.00 -> 35.0 mm, vias 0 -> 1
- net CS: track 0.00 -> 34.0 mm, vias 0 -> 4
- net EN: track 0.00 -> 29.7 mm
- net TX1: track 0.00 -> 28.2 mm, vias 0 -> 2
- net DET: track 0.00 -> 27.4 mm
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- added copper zone on B.Cu, net GND
- added copper zone on F.Cu, net GND
Other:
- board outline added: 51.5 x 76.4 mm

Commit message: Add files via upload
Parts:
- added REF**: MountingHole_4.3mm_M4, MountingHole:MountingHole_4.3mm_M4, F.Cu at (170.5, 89.0)
- added REF**: MountingHole_4.3mm_M4, MountingHole:MountingHole_4.3mm_M4, F.Cu at (117.7, 35.1)
- added REF**: MountingHole_4.3mm_M4, MountingHole:MountingHole_4.3mm_M4, F.Cu at (170.4, 35.1)
- added REF**: MountingHole_4.3mm_M4, MountingHole:MountingHole_4.3mm_M4, F.Cu at (114.9, 89.0)
- BT1: moved to B.Cu
- moved BT1 5.17 mm to (156.1, 30.4), turned to 180 degrees
- moved D7 4.63 mm to (150.5, 28.4)
- moved R10 4.50 mm to (154.5, 28.1), turned to 0 degrees
- moved R7 1.47 mm to (119.1, 40.3)
- moved R11 1.43 mm to (119.1, 41.9)
- moved D2 0.28 mm to (120.7, 41.9)
- moved D6 0.28 mm to (120.7, 40.3)
Routing:
- net VSENS: track 77.2 -> 66.0 mm
- net GND: track 80.6 -> 70.9 mm, vias 84 -> 108
- net Net-(BT1-+): track 10.5 -> 7.29 mm, vias 1 -> 0
- net +3V3: track 145.8 -> 142.8 mm, vias 8 -> 7
- net INT: track 64.1 -> 61.3 mm
- net Net-(D7-K): track 3.19 -> 1.62 mm
- net Net-(D6-K): track 1.42 -> 0.00 mm
- net Net-(D2-K): track 1.39 -> 0.00 mm
- net MOSI: track 49.5 -> 48.9 mm
- net RX1: track 21.1 -> 20.5 mm
Other:
- board size 51.5 x 76.4 mm -> 65 x 67.4 mm

Commit message: Add files via upload
AO3401Aのフットプリントを修正
Parts:
- removed Q4: AO3401A, Package_TO_SOT_SMD:SOT-23
- removed REF** (x4): MountingHole_4.3mm_M4, MountingHole:MountingHole_4.3mm_M4
- added Q1: AO3401A, Package_TO_SOT_SMD:SOT-23, B.Cu at (139.4, 67.3)
- moved C21 2.11 mm to (139.5, 63.8), turned to 90 degrees
Routing:
- net Net-(D20-K): track 20.2 -> 15.0 mm
- net Net-(D20-A): track 8.18 -> 4.64 mm
- net +BATT: track 91.3 -> 90.4 mm
- net GND: vias 108 -> 110

Commit message: Add files via upload
MCP25625のピン19を3V3に変更
Connections:
- C14 pad 1: +5V -> +3V3
- C3 pad 1: +5V -> +3V3
- U3 pad 19: +5V -> +3V3
Routing:
- net +3V3: track 142.8 -> 149.6 mm, vias 7 -> 9
- net +5V: track 26.4 -> 23.4 mm, vias 1 -> 2
- net SCK: vias 4 -> 2
- net GND: vias 110 -> 108
Changed lines of the file:
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@@
 			(layers "F.Cu" "F.Mask" "F.Paste")
 			(roundrect_rratio 0.25)
-			(net 4 "+5V")
+			(net 5 "+3V3")
 			(pinfunction "VDD")
 			(pintype "power_in")
@@
 			(layers "B.Cu" "B.Mask" "B.Paste")
 			(roundrect_rratio 0.25)
-			(net 4 "+5V")
+			(net 5 "+3V3")
 			(pintype "passive")
 		)
@@
 			(layers "B.Cu" "B.Mask" "B.Paste")
 			(roundrect_rratio 0.25)
-			(net 4 "+5V")
+			(net 5 "+3V3")
 			(pintype "passive")
 		)
@@
 	)
 	(via
-		(at 135.7 68)
-		(size 0.5)
-		(drill 0.3)
-		(layers "F.Cu" "B.Cu")
-		(free yes)
-		(net 1)
-	)
-	(via
 		(at 126.7 91.2)
 		(size 0.5)
@@
 	)
 	(via
-		(at 133.03 68.38)
-		(size 0.5)
-		(drill 0.3)
-		(layers "F.Cu" "B.Cu")
-		(free yes)
-		(net 1)
-	)
-	(via
 		(at 135.7 30)
 		(size 0.5)
@@
 	)
 	(segment
-		(start 143.4325 74.3075)
-		(end 139.125 70)
-		(width 0.6)
-		(layer "F.Cu")
-		(net 4)
-	)
-	(segment
-		(start 129.2 68.3)
-		(end 129.2 69.85)
+		(start 144.05 69.6)
+		(end 142.61 68.16)
 		(width 0.4)
 		(layer "F.Cu")
@@
 	)
 	(segment
-		(start 129.2 69.85)
-		(end 129.35 70)
+		(start 142.61 68.16)
+		(end 137.71 68.16)
 		(width 0.4)
 		(layer "F.Cu")
 		(net 4)
 	)
-	(segment
-		(start 139.125 70)
-		(end 129.35 70)
-		(width 0.6)
-		(layer "F.Cu")
+	(via
+		(at 137.71 68.16)
+		(size 0.7)
+		(drill 0.5)
+		(layers "F.Cu" "B.Cu")
 		(net 4)
 	)
 	(via
-		(at 129.35 70)
+		(at 144.05 69.6)
 		(size 0.7)
 		(drill 0.5)
@@
 	)
 	(segment
-		(start 144.05 69.6)
-		(end 144.05 70.35)
-		(width 0.6)
+		(start 129.24 68.16)
+		(end 127.5 69.9)
+		(width 0.4)
 		(layer "B.Cu")
 		(net 4)
 	)
 	(segment
-		(start 129.35 70)
-		(end 127.6 70)
-		(width 0.4)
+		(start 144.05 69.6)
+		(end 144.05 70.35)
+		(width 0.6)
 		(layer "B.Cu")
 		(net 4)
 	)
 	(segment
-		(start 129.35 70)
-		(end 129.35 71.5)
+		(start 137.71 68.16)
+		(end 129.24 68.16)
 		(width 0.4)
 		(layer "B.Cu")
@@
 	)
 	(segment
+		(start 129.35 70)
+		(end 129.2 69.85)
+		(width 0.4)
+		(layer "F.Cu")
+		(net 5)
+	)
+	(segment
 		(start 137.3 51.2875)
 		(end 137.3 53.525)
@@
 	)
 	(segment
+		(start 129.2 68.3)
+		(end 129.2 67.288708)
+		(width 0.4)
+		(layer "F.Cu")
+		(net 5)
+	)
+	(segment
+		(start 127.511292 65.6)
+		(end 127.35 65.6)
+		(width 0.4)
+		(layer "F.Cu")
+		(net 5)
+	)
+	(segment
 		(start 139.5 47.5)
 		(end 139.5 49.0875)
@@
 	)
 	(segment
+		(start 129.2 69.85)
+		(end 129.2 68.3)
+		(width 0.4)
+		(layer "F.Cu")
+		(net 5)
+	)
+	(segment
 		(start 143.12 51.12)
 		(end 141 49)
@@
 	)
 	(segment
+		(start 129.2 67.288708)
+		(end 127.511292 65.6)
+		(width 0.4)
+		(layer "F.Cu")
+		(net 5)
+	)
+	(segment
 		(start 153.5 31.1)
 		(end 156.58 34.18)
@@
 	)
 	(via
+		(at 129.35 70)
+		(size 0.7)
+		(drill 0.5)
+		(layers "F.Cu" "B.Cu")
+		(net 5)
+	)
+	(via
 		(at 141 49)
 		(size 0.7)
@@
 	)
 	(via
+		(at 127.35 65.6)
+		(size 0.7)
+		(drill 0.5)
+		(layers "F.Cu" "B.Cu")
+		(net 5)
+	)
+	(via
 		(at 123.2 29.21)
 		(size 0.7)
@@
 	)
 	(segment
+		(start 129.35 71.5)
+		(end 129.35 70)
+		(width 0.4)
+		(layer "B.Cu")
+		(net 5)
+	)
+	(segment
 		(start 126.3 29.475)
 		(end 124.8 29.475)
@@
 	)
 	(segment
-		(start 136.59 61.194942)
-		(end 138.9 58.884942)
+		(start 138.9 58.884942)
+		(end 136.59 61.194942)
 		(width 0.4)
 		(layer "F.Cu")
@@
 	)
 	(segment
-		(start 131.8 75.3)
-		(end 134.3435 72.7565)
+		(start 136.215812 55.945)
+		(end 136.55 55.610812)
 		(width 0.4)
 		(layer "F.Cu")
@@
 	)
 	(segment
-		(start 136.215812 55.945)
-		(end 136.55 55.610812)
+		(start 136.59 70.51)
+		(end 131.8 75.3)
 		(width 0.4)
 		(layer "F.Cu")
@@
 	)
 	(segment
-		(start 136.59 64.6)
-		(end 136.59 61.194942)
+		(start 138.9 53.255484)
+		(end 138.9 58.884942)
 		(width 0.4)
 		(layer "F.Cu")
@@
 	)
 	(segment
-		(start 138.9 58.884942)
-		(end 138.9 53.255484)
+		(start 136.59 61.194942)
+		(end 136.59 70.51)
 		(width 0.4)
 		(layer "F.Cu")
@@
 	)
 	(via
-		(at 134.3435 72.7565)
-		(size 0.7)
-		(drill 0.5)
-		(layers "F.Cu" "B.Cu")
-		(net 38)
-	)
-	(via
 		(at 138.9 53.255484)
 		(size 0.7)
@@
 		(net 38)
 	)
-	(via
-		(at 136.59 64.6)
-		(size 0.7)
-		(drill 0.5)
-		(layers "F.Cu" "B.Cu")
-		(net 38)
-	)
-	(segment
-		(start 134.3435 66.8565)
-		(end 134.3435 72.7565)
-		(width 0.4)
-		(layer "B.Cu")
-		(net 38)
-	)
 	(segment
 		(start 138.251 40.668516)
@@
 		(width 0.4)
 		(layer "B.Cu")
-		(net 38)
-	)
-	(segment
-		(start 134.3435 66.8565)
-		(end 136.59 64.61)
-		(width 0.4)
-		(layer "B.Cu")
-		(net 38)
-	)
-	(segment
-		(start 136.59 64.61)
-		(end 136.59 64.6)
-		(width 0.4)
-		(layer "B.Cu")

Commit message: Add files via upload
MCP25625 ピン19を3V3に変更。取付穴を追加。
Parts:
- added REF**: MountingHole_3.5mm, MountingHole:MountingHole_3.5mm, F.Cu at (170.7, 89.0)
- added REF**: MountingHole_3.5mm, MountingHole:MountingHole_3.5mm, F.Cu at (170.7, 34.8)
- added REF**: MountingHole_3.5mm, MountingHole:MountingHole_3.5mm, F.Cu at (115.6, 89.0)
- added REF**: MountingHole_3.5mm, MountingHole:MountingHole_3.5mm, F.Cu at (117.2, 34.8)
