File: MainBoard2026/MainBoard2026.kicad_sch (KiCad schematic)
At the start: 73 parts, among them J1 RJ25, J2 RJ25, J4 RJ25, J5 GPS_DFROBOT_TEL-0157, J6 Micro_SD_Card_Det_Hirose_DM3AT, J8 BATT_CON, Q4 AO3401A, SW3 POWER, U1 ESP32-WROOM-32, U2 R-78E5.0-0.5, U3 MCP25625-x-SS, U4 R-78E3.3-0.5, U6 RX8900_mod, Y1 16MHz

Commit message: Add files via upload
Parts:
- removed D8: SPI, LED_SMD:LED_0603_1608Metric, symbol Device:LED
- removed R20: 22, Resistor_SMD:R_0603_1608Metric, symbol Device:R_US
- removed R21: 33, Resistor_SMD:R_0603_1608Metric, symbol Device:R_US
- added D2: ERR2, LED_SMD:LED_0603_1608Metric, symbol Device:LED
- added J3: ICSP, Connector_PinHeader_2.54mm:PinHeader_2x03_P2.54mm_Vertical, symbol Connector:Conn_01x06_Socket
- added R13: 10k, Resistor_SMD:R_0603_1608Metric, symbol Device:R_US
- C5: footprint Capacitor_SMD:C_1206_3216Metric -> Capacitor_SMD:C_0603_1608Metric
- D20: value Zener_10V -> Zener_9V1; footprint Diode_SMD:D_SOD-323 -> KUBTSS:Zenner
- D4: value SCK -> SD
- D5: value ERR -> CAN
- D6: value BATT -> ERR
- R5, R6: value 1k -> 2k
- U1: footprint RF_Module:ESP32-WROOM-32 -> KUBTSS:ESP32-WROOM-32
- U4: value R-78E3.3-0.5 -> BP5293-33; footprint Converter_DCDC:Converter_DCDC_RECOM_R-78E-0.5_THT -> KUBTSS:BP5293-33
Connections:
- net +3.3V is gone; now on net +3V3: C28.2, C29.2, D9.2 (A), U4.3 (OUT)
- net +out is gone; now on net +BATT: Q4.2 (D)
- net LED2 is gone; now on net ERR: U1.11 (IO26)
- net +3V3: now also D4.2 (A), D5.2 (A), J5.1 (Pin_1), R25.2, J3.6 (Pin_6)
- net +5V: no longer J5.1 (Pin_1)
- net CS: now also R6.2, U1.23 (IO15), U3.17 (~{CS})
- net CS1: now also R5.2
- net DET: now also U1.6 (IO34); no longer U1.36 (IO22)
- net EN: now also J3.5 (Pin_5)
- net ERR: now also D6.2 (A); no longer D5.2 (A), U1.7 (IO35)
- net GND: now also J3.2 (Pin_2), R13.2; no longer R25.2, R5.2, R6.2
- net INT: now also U1.26 (IO4); no longer U1.8 (IO32)
- net IO0: now also J3.3 (Pin_3)
- net MISO: now also U1.31 (IO19); no longer U1.33 (IO21)
- net RX: now also J3.4 (Pin_4)
- net SCL: now also U1.36 (IO22); no longer U1.13 (IO14)
- net SDA: now also U1.33 (IO21); no longer U1.23 (IO15)
- net TX: now also J3.1 (Pin_1)
- net TX1: now also R25.1, U1.28 (IO17); no longer U1.12 (IO27)
- net at C7.1, R27.2: now also U1.7 (IO35); no longer U1.29 (IO5)
- net at R11.1: now also D2.1 (K)
- net at R31.1: now also U1.37 (IO23); no longer U1.30 (IO18)
- net at U1.14 (IO12): now also R13.1
- net at R30.1: now also U1.29 (IO5); no longer U1.28 (IO17)
- net at R32.1: now also U1.30 (IO18); no longer U1.31 (IO19)
- removed net BAT: D6.2 (A), U1.6 (IO34)
- net LED1: no longer names the net of U1.10 (IO25)
- net LED1: no longer D4.2 (A)
- new net ERR2: D2.2 (A), U1.12 (IO27)
Other:
- note added: "I2C SDA:IO21,SCL:IO22 SPI SCK:IO18,MISO:IO19,MOSI:IO23,CS:IO5, CS2:IO15 UART0(書き込み） TX:IO1,RX:IO3 UART1(未接続） UART2(外部機器） TX:IO17,RX16"
- moved on the sheet: C7, D4, D5, D6, JP1, R25, R27, R30, R31, R32, R5, R6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

Commit message: Add files via upload
Connections:
- net GND: now also U3.26 (VSS)
Changed lines of the file:
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@@
 	)
 	(junction
+		(at 200.66 306.07)
+		(diameter 0)
+		(color 0 0 0 0)
+	)
+	(junction
 		(at 68.58 73.66)
 		(diameter 0)
@@
 	(wire
 		(pts
+			(xy 208.28 304.8) (xy 208.28 306.07)
+		)
+		(stroke
+			(width 0)
+			(type default)
+		)
+	)
+	(wire
+		(pts
 			(xy 218.44 245.11) (xy 224.79 245.11)
 		)
@@
 	(wire
 		(pts
-			(xy 200.66 304.8) (xy 200.66 309.88)
+			(xy 200.66 304.8) (xy 200.66 306.07)
 		)
 		(stroke
@@
 	(wire
 		(pts
+			(xy 208.28 306.07) (xy 200.66 306.07)
+		)
+		(stroke
+			(width 0)
+			(type default)
+		)
+	)
+	(wire
+		(pts
 			(xy 142.24 22.86) (xy 149.86 22.86)
 		)
@@
 	(wire
 		(pts
+			(xy 200.66 306.07) (xy 200.66 309.88)
+		)
+		(stroke
+			(width 0)
+			(type default)
+		)
+	)
+	(wire
+		(pts
 			(xy 73.66 73.66) (xy 73.66 80.01)
 		)
@@
 		)
 		(property "Value" "+5V"
-			(at 77.47 13.97 0)
+			(at 80.01 17.7799 0)
 			(effects
 				(font
 					(size 1.27 1.27)
 				)
+				(justify left)
 			)
 		)
